File: gpio_v2/gpio_v2.kicad_pcb (KiCad board)
At the start: 2 copper layers, 85 x 56 mm, 37 parts, among them J3 Raspberry_Pi_2_3, M25 GND_25, M30 GND_30, M34 GND_34, M39 GND_39

Commit message: Add files via upload
Routing:
- net Net-(G0-Pin_1): track 402.0 -> 416.4 mm
- net Net-(G4-Pin_1): track 360.1 -> 370.2 mm
- net Net-(G8-Pin_1): track 208.4 -> 217.8 mm
- net Net-(G22-Pin_1): track 153.5 -> 155.5 mm
- net Net-(G15-Pin_1): track 61.1 -> 62.9 mm
- net Net-(G12-Pin_1): track 62.3 -> 63.8 mm
- net Net-(G13-Pin_1): track 60.4 -> 61.3 mm
- net Net-(G3-Pin_1): track 177.1 -> 177.9 mm
- net Net-(2-V3-Pin_2): track 193.7 -> 194.4 mm
